File: esp32-watering.kicad_pcb (KiCad board)
At the start: 2 copper layers, 25 parts, among them J1 5V, J2 12V, J3 Water Level, J4 Pump, J5 Zone 1, J6 Zone 2, J7 Zone 3, K1 Pump Control, K2 Zone 1, K3 Zone 2, K4 Zone 3, Q1 2N3904, Q2 2N3904, Q3 2N3904, Q4 2N3904, U1 esp32-wemos-d1-mini

Commit message: Start layout
Parts:
- J1, J2: footprint Connector_JST:JST_XH_S2B-XH-A-1_1x02_P2.50mm_Horizontal -> Connector_JST:JST_XH_B2B-XH-A_1x02_P2.50mm_Vertical
- moved U1 122.3 mm to (241.6, 75.1)
- moved K4 92.3 mm to (152.0, 51.2), turned to 180 degrees
- moved K3 80.2 mm to (152.0, 65.0), turned to 180 degrees
- moved K1 79.6 mm to (152.0, 93.0), turned to 180 degrees
- moved K2 75.5 mm to (152.0, 79.0), turned to 180 degrees
- moved R5 66.7 mm to (177.0, 52.8), turned to 90 degrees
- moved J3 62.2 mm to (140.0, 105.5), turned to 180 degrees
- moved J7 61.0 mm to (140.1, 53.7), turned to 180 degrees
- moved Q4 53.0 mm to (171.6, 55.0), turned to 180 degrees
- moved J4 51.9 mm to (140.0, 95.7), turned to 180 degrees
- moved D4 51.0 mm to (164.5, 46.3), turned to -90 degrees
- moved R4 50.8 mm to (177.0, 66.8), turned to 90 degrees
- moved R1 50.4 mm to (148.0, 105.5)
- moved J6 49.4 mm to (140.0, 67.6), turned to 180 degrees
- moved J1 47.8 mm to (239.1, 46.1), turned to 180 degrees
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
Commit message: More layout
Parts:
- moved U1 144.9 mm to (96.7, 73.4)
- moved J1 140.1 mm to (99.0, 44.2), turned to 0 degrees
- moved J2 139.8 mm to (90.3, 44.2), turned to 0 degrees
- moved J4 83.9 mm to (191.5, 29.5), turned to 0 degrees
- moved R5 71.5 mm to (228.2, 102.7), turned to 0 degrees
- moved Q1 70.1 mm to (159.4, 27.5), turned to 0 degrees
- moved K1 66.7 mm to (179.5, 32.2), turned to 0 degrees
- moved J5 64.1 mm to (191.5, 43.5), turned to 0 degrees
- moved R4 61.2 mm to (228.2, 100.3), turned to 0 degrees
- moved J3 55.4 mm to (191.2, 84.3), turned to 0 degrees
- moved J7 54.2 mm to (191.4, 71.5), turned to 0 degrees
- moved J6 52.4 mm to (191.5, 57.6), turned to 0 degrees
- moved D1 50.2 mm to (167.0, 37.5), turned to 90 degrees
- moved Q2 43.0 mm to (159.5, 41.4), turned to 0 degrees
- moved K2 42.8 mm to (179.5, 46.2), turned to 0 degrees
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Routing:
- net Net-(D1-A): track 0.00 -> 15.3 mm

Commit message: Indicative layout
Parts:
- moved R5 87.2 mm to (146.2, 73.0)
- moved R4 85.5 mm to (146.2, 76.0)
- moved R3 65.7 mm to (146.2, 79.0)
- moved R2 63.9 mm to (146.2, 82.0)
- moved U1 52.9 mm to (140.6, 43.9)
- moved J1 50.8 mm to (130.0, 84.5), turned to 90 degrees
- moved J2 50.2 mm to (130.0, 75.0), turned to 90 degrees
- moved R1 29.0 mm to (146.2, 85.0)
- moved J3 2.89 mm to (194.0, 85.0), turned to 180 degrees

Commit message: Initial layout
Parts:
- moved J3 34.6 mm to (161.0, 74.5), turned to -90 degrees
- moved R2 16.7 mm to (153.6, 67.0), turned to 180 degrees
- moved R3 12.1 mm to (153.6, 69.5), turned to 180 degrees
- moved J1 10.5 mm to (130.8, 74.0), turned to 180 degrees
- moved J2 10.0 mm to (140.0, 74.0), turned to 180 degrees
- moved R4 8.44 mm to (153.6, 72.0), turned to 180 degrees
- moved R1 8.00 mm to (146.0, 77.0)
- moved R5 7.58 mm to (153.6, 74.5), turned to 180 degrees
- moved J5 3.57 mm to (192.0, 47.0), turned to 90 degrees
- moved J4 3.29 mm to (192.0, 32.8), turned to 90 degrees
- moved J6 2.91 mm to (192.0, 60.5), turned to 90 degrees
- moved J7 2.59 mm to (192.0, 74.0), turned to 90 degrees
- moved U1 2.25 mm to (138.6, 44.9)
- moved K4 1.20 mm to (179.5, 72.8)
- moved K3 1.01 mm to (179.4, 59.2)
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Connections:
- U1 pad 16: unconnected-(U1-3V3-Pad16) -> +3.3V
Routing:
- net +12V: track 0.00 -> 208.1 mm
- net Net-(Q1-B): track 0.00 -> 41.9 mm
- net +5V: track 0.00 -> 31.8 mm
- net Net-(Q2-B): track 0.00 -> 31.0 mm
- net Net-(Q3-B): track 0.00 -> 19.8 mm
- net Net-(D2-A): track 0.00 -> 14.8 mm
- net Net-(D3-A): track 0.00 -> 14.7 mm
- net Net-(D4-A): track 0.00 -> 14.7 mm
- net Net-(Q4-B): track 0.00 -> 10.9 mm
- net Net-(J3-Pin_2): track 0.00 -> 7.38 mm
- net Net-(J5-Pin_2): track 0.00 -> 7.24 mm
- net Net-(J6-Pin_2): track 0.00 -> 7.15 mm
- net Net-(J4-Pin_2): track 0.00 -> 7.06 mm
- net Net-(J7-Pin_2): track 0.00 -> 7.04 mm
- added copper zone on B.Cu, net GND
Other:
- board outline added: 75 x 55.5 mm
- board text added: "ESP32 House Plant Watering Controller Rev 1.1"

Commit message: Flip float valve
Parts:
- J3: value Water Level -> Float
Connections:
- J3 pad 1: +3.3V -> Net-(J3-Pin_1)
- J3 pad 2: Net-(J3-Pin_2) -> +3.3V
- R1 pad 2: Net-(J3-Pin_2) -> Net-(J3-Pin_1)
- U1 pad 24: Net-(J3-Pin_2) -> Net-(J3-Pin_1)
Routing:
- net +3.3V: track 0.00 -> 73.6 mm
- net Net-(U1-IO_17/D3): track 0.00 -> 33.7 mm
- net Net-(J3-Pin_1): track 0.00 -> 8.42 mm
- net Net-(J3-Pin_2): track 7.38 -> 0.00 mm
Changed lines of the file:
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@@
 	(net 7 "GND")
 	(net 8 "+3.3V")
-	(net 9 "Net-(J3-Pin_2)")
+	(net 9 "Net-(J3-Pin_1)")
 	(net 10 "Net-(J4-Pin_2)")
 	(net 11 "Net-(J5-Pin_2)")
@@
 			(layers "*.Cu" "*.Mask")
 			(remove_unused_layers no)
-			(net 9 "Net-(J3-Pin_2)")
+			(net 9 "Net-(J3-Pin_1)")
 			(pinfunction "IO_27")
 			(pintype "bidirectional")
@@
 			(layers "*.Cu" "*.Mask")
 			(remove_unused_layers no)
-			(net 9 "Net-(J3-Pin_2)")
+			(net 9 "Net-(J3-Pin_1)")
 			(pintype "passive")
 		)
@@
 			)
 		)
-		(property "Value" "Water Level"
+		(property "Value" "Float"
 			(at 1 3 90)
 			(layer "B.SilkS")
@@
 			(remove_unused_layers no)
 			(roundrect_rratio 0.147059)
-			(net 8 "+3.3V")
+			(net 9 "Net-(J3-Pin_1)")
 			(pinfunction "Pin_1")
 			(pintype "passive")
@@
 			(layers "*.Cu" "*.Mask")
 			(remove_unused_layers no)
-			(net 9 "Net-(J3-Pin_2)")
+			(net 8 "+3.3V")
 			(pinfunction "Pin_2")
 			(pintype "passive")
@@
 	)
 	(segment
+		(start 125.45 79.4)
+		(end 122.751 76.701)
+		(width 0.5)
+		(layer "F.Cu")
+		(net 8)
+	)
+	(segment
+		(start 158.55 79.45)
+		(end 125.45 79.45)
+		(width 0.5)
+		(layer "F.Cu")
+		(net 8)
+	)
+	(segment
+		(start 125.45 79.45)
+		(end 125.45 79.4)
+		(width 0.5)
+		(layer "F.Cu")
+		(net 8)
+	)
+	(segment
+		(start 122.751 76.701)
+		(end 122.751 68.65)
+		(width 0.5)
+		(layer "F.Cu")
+		(net 8)
+	)
+	(segment
 		(start 161 77)
+		(end 158.55 79.45)
+		(width 0.5)
+		(layer "F.Cu")
+		(net 8)
+	)
+	(segment
+		(start 129.73 51.28)
+		(end 127.14 51.28)
+		(width 0.5)
+		(layer "F.Cu")
+		(net 8)
+	)
+	(segment
+		(start 132.5 54.05)
+		(end 129.73 51.28)
+		(width 0.5)
+		(layer "F.Cu")
+		(net 8)
+	)
+	(segment
+		(start 122.751 68.65)
+		(end 132.5 58.901)
+		(width 0.5)
+		(layer "F.Cu")
+		(net 8)
+	)
+	(segment
+		(start 132.5 58.901)
+		(end 132.5 54.05)
+		(width 0.5)
+		(layer "F.Cu")
+		(net 8)
+	)
+	(segment
+		(start 161 74.5)
+		(end 158.5 77)
+		(width 0.5)
+		(layer "F.Cu")
+		(net 9)
+	)
+	(segment
+		(start 158.5 77)
 		(end 153.62 77)
 		(width 0.5)
@@
 		(net 17)
 	)
+	(segment
+		(start 146.39 43.66)
+		(end 150 43.66)
+		(width 0.5)
+		(layer "F.Cu")
+		(net 19)
+	)
+	(segment
+		(start 146 69.5)
+		(end 141.05 64.55)
+		(width 0.5)
+		(layer "F.Cu")
+		(net 19)
+	)
+	(segment
+		(start 141.05 64.55)
+		(end 141.05 49)
+		(width 0.5)
+		(layer "F.Cu")
+		(net 19)
+	)
+	(segment
+		(start 141.05 49)
+		(end 146.39 43.66)
+		(width 0.5)
+		(layer "F.Cu")
+		(net 19)
+	)
 	(zone
 		(net 7)
@@
 		(polygon
 			(pts
-				(xy 122.5 25.5) (xy 196 25.5) (xy 196.471966 76.000377) (xy 122.972357 76.986949)
+				(xy 122 25.5) (xy 196.5 25.5) (xy 197.005174 79.553624) (xy 122.505078 80.553626)
 			)
 		)

Commit message: Pre-DRC
Parts:
- added ?: , , F.Cu at (126.3, 66.5)
- added ?: , , F.Cu at (192.2, 67.0)
- added REF**: MountingHole_2.5mm_Pad_TopOnly, MountingHole:MountingHole_2.5mm_Pad_TopOnly, F.Cu at (126.3, 66.5)
- added REF**: MountingHole_2.5mm_Pad_TopOnly, MountingHole:MountingHole_2.5mm_Pad_TopOnly, F.Cu at (192.2, 67.0)
- added REF**: MountingHole_2.5mm_Pad_TopOnly, MountingHole:MountingHole_2.5mm_Pad_TopOnly, F.Cu at (161.6, 34.5)
- moved R2 32.3 mm to (156.5, 34.8), turned to -90 degrees
- moved R3 21.2 mm to (156.4, 48.5), turned to -90 degrees
- moved R4 10.2 mm to (156.4, 62.1), turned to -90 degrees
- moved J7 1.55 mm to (192.0, 75.5)
- moved R5 1.55 mm to (153.6, 73.0)
- moved J6 1.45 mm to (192.0, 59.0)
- moved R1 1.40 mm to (146.0, 75.6)
- moved U1 0.67 mm to (137.9, 45.0)
- moved Q3 0.16 mm to (159.5, 55.0)
- moved Q1 0.10 mm to (159.4, 28.1)
- moved Q4 0.10 mm to (159.6, 68.7)
- moved J2 0.10 mm to (139.9, 74.0)
- moved J1 0.06 mm to (130.8, 74.0)
- moved Q2 0.05 mm to (159.4, 41.4)
Connections:
- R2 pad 2: Net-(U1-IO_12/TDI) -> Net-(U1-IO_27)
- R3 pad 2: Net-(U1-IO_17/D3) -> Net-(U1-IO_32)
- R4 pad 2: Net-(U1-IO_32) -> Net-(U1-IO_12/TDI)
- R5 pad 2: Net-(U1-IO_25) -> Net-(U1-IO_17/D3)
- U1 pad 24: Net-(J3-Pin_1) -> Net-(U1-IO_27)
- U1 pad 26: Net-(U1-IO_25) -> unconnected-(U1-IO_25-Pad26)
- U1 pad 31: unconnected-(U1-IO_16/D4-Pad31) -> Net-(J3-Pin_1)
Routing:
- net Net-(Q1-B): track 41.9 -> 8.73 mm
- net Net-(J3-Pin_1): track 8.42 -> 40.9 mm
- net Net-(U1-IO_12/TDI): track 0.00 -> 27.7 mm
- net Net-(Q2-B): track 31.0 -> 9.24 mm
- net Net-(U1-IO_32): track 0.00 -> 17.5 mm
- net Net-(Q3-B): track 19.8 -> 9.24 mm
- net Net-(U1-IO_27): track 0.00 -> 9.32 mm
- net +12V: track 208.1 -> 209.9 mm
- net +3.3V: track 73.6 -> 72.0 mm
- net Net-(U1-IO_17/D3): track 33.7 -> 32.2 mm
- net Net-(Q4-B): track 10.9 -> 9.71 mm
- net Net-(J7-Pin_2): track 7.04 -> 7.65 mm
- net Net-(J6-Pin_2): track 7.15 -> 6.55 mm

Commit message: Pass DRC
Parts:
- removed ? (x2): , 
- J3: value Float -> FLOAT
- J4: value Pump -> PUMP
- J5: value Zone 1 -> ZONE 1
- J6: value Zone 2 -> ZONE 2
- J7: value Zone 3 -> ZONE 3
- moved REF** 0.91 mm to (127.2, 66.3)
Routing:
- net Net-(J3-Pin_1): track 40.9 -> 41.4 mm
Changed lines of the file:
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@@
 	(footprint "MountingHole:MountingHole_2.5mm_Pad_TopOnly"
 		(layer "F.Cu")
-		(at 126.35 66.45)
+		(at 127.25 66.3)
 		(descr "Mounting Hole 2.5mm, generated by kicad-footprint-generator mountinghole.py")
 		(tags "mountinghole")
@@
 			)
 		)
-		(property "Value" "Zone 2"
+		(property "Value" "ZONE 2"
 			(at -4.15 0.45 180)
 			(layer "F.SilkS")
@@
 			)
 		)
-		(property "Value" "Pump"
+		(property "Value" "PUMP"
 			(at -4.3 0.5 180)
 			(layer "F.SilkS")
@@
 			)
 		)
-		(property "Value" "Zone 3"
+		(property "Value" "ZONE 3"
 			(at -3.95 0.7 180)
 			(layer "F.SilkS")
@@
 		(attr through_hole)
 		(fp_line
-			(start -16.25 -16.51)
-			(end -16.25 12.7)
+			(start -16.275 12.95)
+			(end -12.725 12.95)
 			(stroke
 				(width 0.12)
@@
 		)
 		(fp_line
-			(start -16.25 12.7)
-			(end -12.7 12.7)
+			(start -16.25 -16.51)
+			(end -16.275 12.95)
 			(stroke
 				(width 0.12)
@@
 		)
 		(fp_line
-			(start -12.7 12.7)
+			(start -12.7 12.95)
 			(end -12.7 17.78)
 			(stroke
@@
 			)
 		)
-		(property "Value" "Float"
+		(property "Value" "FLOAT"
 			(at 1.05 5.05 90)
 			(layer "F.SilkS")
@@
 			)
 		)
-		(property "Value" "Zone 1"
+		(property "Value" "ZONE 1"
 			(at -4.35 0.45 180)
 			(layer "F.SilkS")
@@
 			(at 0 3.45 0)
 			(layer "F.Fab")
+			(hide yes)
 			(effects
 				(font
@@
 		(embedded_fonts no)
 	)
-	(footprint ""
-		(layer "F.Cu")
-		(at 126.35 66.45)
-		(property "Reference" ""
-			(at 0 0 0)
-			(layer "F.SilkS")
-			(effects
-				(font
-					(size 1.27 1.27)
-					(thickness 0.15)
-				)
-			)
-		)
-		(property "Value" ""
-			(at 0 0 0)
-			(layer "F.Fab")
-			(effects
-				(font
-					(size 1.27 1.27)
-					(thickness 0.15)
-				)
-			)
-		)
-		(property "Datasheet" ""
-			(at 0 0 0)
-			(layer "F.Fab")
-			(hide yes)
-			(effects
-				(font
-					(size 1.27 1.27)
-					(thickness 0.15)
-				)
-			)
-		)
-		(property "Description" ""
-			(at 0 0 0)
-			(layer "F.Fab")
-			(hide yes)
-			(effects
-				(font
-					(size 1.27 1.27)
-					(thickness 0.15)
-				)
-			)
-		)
-		(pad "1" connect circle
-			(at 0 0)
-			(size 5.6 5.6)
-			(layers "F.Cu" "F.Mask")
-			(zone_connect 2)
-		)
-		(embedded_fonts no)
-	)
 	(footprint "MountingHole:MountingHole_2.5mm_Pad_TopOnly"
 		(layer "F.Cu")
@@
 		)
 	)
-	(footprint ""
-		(layer "F.Cu")
-		(at 192.25 66.95)
-		(property "Reference" ""
-			(at 0 0 0)
-			(layer "F.SilkS")
-			(effects
-				(font
-					(size 1.27 1.27)
-					(thickness 0.15)
-				)
-			)
-		)
-		(property "Value" ""
-			(at 0 0 0)
-			(layer "F.Fab")
-			(effects
-				(font
-					(size 1.27 1.27)
-					(thickness 0.15)
-				)
-			)
-		)
-		(property "Datasheet" ""
-			(at 0 0 0)
-			(layer "F.Fab")
-			(hide yes)
-			(effects
-				(font
-					(size 1.27 1.27)
-					(thickness 0.15)
-				)
-			)
-		)
-		(property "Description" ""
-			(at 0 0 0)
-			(layer "F.Fab")
-			(hide yes)
-			(effects
-				(font
-					(size 1.27 1.27)
-					(thickness 0.15)
-				)
-			)
-		)
-		(pad "1" thru_hole circle
-			(at 0 0)
-			(size 2.9 2.9)
-			(drill 2.5)
-			(layers "*.Cu" "*.Mask")
-			(remove_unused_layers no)
-			(zone_connect 2)
-		)
-		(embedded_fonts no)
-	)
 	(footprint "SR5-12V-200-1C:RELAY_SR5-12V-200-1C"
 		(layer "F.Cu")
@@
 	)
 	(gr_rect
-		(start 134 38)
-		(end 142 56)
+		(start 133.9 36)
+		(end 141.9 54)
 		(stroke
 			(width 0.1)
@@
 	)
 	(gr_text "ESP32 House Plant \nWatering Controller\nRev 1.1"
-		(at 138 47 90)
+		(at 137.9 45 90)
 		(layer "B.SilkS")
 		(effects
 			(font
 				(size 1 1)
-				(thickness 0.1)
+				(thickness 0.15)
 			)
 			(justify mirror)
@@
 	)
 	(segment
+		(start 146.85 51.35)
+		(end 132.4 65.8)
+		(width 1.5)
+		(layer "B.Cu")
+		(net 6)
+	)
+	(segment
 		(start 149.33 51.35)
 		(end 146.85 51.35)
@@
 	)
 	(segment
-		(start 130.75 67.45)
-		(end 146.85 51.35)
+		(start 132.4 65.8)
+		(end 132.4 72.375)
 		(width 1.5)
 		(layer "B.Cu")
@@
 	)
 	(segment
-		(start 130.75 67.45)
+		(start 132.4 72.375)
 		(end 130.75 74.025)
 		(width 1.5)
@@
 	(segment
 		(start 146.681 68.671)
-		(end 146.681 48.344844)
+		(end 146.681 47.469)
 		(width 0.5)
 		(layer "F.Cu")
@@
 	)
 	(segment
-		(start 153.61 75.6)
-		(end 146.681 68.671)
+		(start 146.681 47.469)
+		(end 147.88 46.27)
 		(width 0.5)
 		(layer "F.Cu")
@@
 	)
 	(segment
-		(start 146.681 48.344844)
+		(start 147.88 46.27)
 		(end 148.755844 46.27)
 		(width 0.5)
 		(layer "F.Cu")
+		(net 9)
+	)
+	(segment
+		(start 153.61 75.6)
+		(end 146.681 68.671)
+		(width 0.5)
+		(layer "F.Cu")
