File: esp32-watering.kicad_pcb (KiCad board)
At the start: 2 copper layers, 75 x 55.5 mm, 30 parts, among them J1 12V, J2 DS18B20, J3 Water Level, J4 Pump, J5 Zone 1, J6 Zone 2, J7 Zone 3, K1 Pump Control, K2 Zone 1, K3 Zone 2, K4 Zone 3, Q1 2N3904, Q2 2N3904, Q3 2N3904, Q4 2N3904, U1 esp32-wemos-d1-mini, U2 TSR 1-2433

Commit message: Change silkscreen, refill zones
Parts:
- J3: value Water Level -> FLOAT
- J4: value Pump -> PUMP
- J5: value Zone 1 -> ZONE 1
- J6: value Zone 2 -> ZONE 2
- J7: value Zone 3 -> ZONE 3
- moved REF** 0.14 mm to (161.7, 34.6)
Other:
- board size 75 x 55.5 mm -> 74.7 x 55.5 mm
Changed lines of the file:
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@@
 			(at 3.77 0.05 90)
 			(layer "F.SilkS")
+			(hide yes)
 			(effects
 				(font
@@
 		)
 		(property "Value" "4K7"
-			(at 3.81 1.92 90)
-			(layer "F.Fab")
+			(at 3.81 0 90)
+			(layer "F.SilkS")
 			(effects
 				(font
@@
 			(at 3.81 0 90)
 			(layer "F.SilkS")
+			(hide yes)
 			(effects
 				(font
@@
 		)
 		(property "Value" "1K6"
-			(at 3.81 1.92 90)
-			(layer "F.Fab")
+			(at 3.81 0 90)
+			(layer "F.SilkS")
 			(effects
 				(font
@@
 			)
 		)
-		(property "Value" "Zone 2"
+		(property "Value" "ZONE 2"
 			(at -4.15 0.45 180)
 			(layer "F.SilkS")
@@
 			)
 		)
-		(property "Value" "Pump"
+		(property "Value" "PUMP"
 			(at -4.3 0.5 180)
 			(layer "F.SilkS")
@@
 			)
 		)
-		(property "Value" "Zone 3"
+		(property "Value" "ZONE 3"
 			(at -3.95 0.7 180)
 			(layer "F.SilkS")
@@
 			(at 3.81 0 90)
 			(layer "F.SilkS")
+			(hide yes)
 			(effects
 				(font
@@
 		)
 		(property "Value" "1K6"
-			(at 3.81 1.92 90)
-			(layer "F.Fab")
+			(at 3.81 0 90)
+			(layer "F.SilkS")
 			(effects
 				(font
@@
 			(at 5.08 0 90)
 			(layer "F.SilkS")
+			(hide yes)
 			(effects
 				(font
@@
 		(property "Value" "1N4004"
 			(at 5.08 2.47 90)
-			(layer "F.Fab")
+			(layer "F.SilkS")
 			(effects
 				(font
@@
 			(at 5.08 0 90)
 			(layer "F.SilkS")
+			(hide yes)
 			(effects
 				(font
@@
 		(property "Value" "1N4004"
 			(at 5.08 2.47 90)
-			(layer "F.Fab")
+			(layer "F.SilkS")
 			(effects
 				(font
@@
 			(at 3.81 0 90)
 			(layer "F.SilkS")
+			(hide yes)
 			(effects
 				(font
@@
 		)
 		(property "Value" "1K6"
-			(at 3.81 1.92 90)
-			(layer "F.Fab")
+			(at 3.81 0 90)
+			(layer "F.SilkS")
 			(effects
 				(font
@@
 			(at 3.81 0 90)
 			(layer "F.SilkS")
+			(hide yes)
 			(effects
 				(font
@@
 		)
 		(property "Value" "1K6"
-			(at 3.81 1.92 90)
-			(layer "F.Fab")
+			(at 3.81 0 90)
+			(layer "F.SilkS")
 			(effects
 				(font
@@
 			(at 3.81 0 90)
 			(layer "F.SilkS")
+			(hide yes)
 			(effects
 				(font
@@
 		)
 		(property "Value" "10K"
-			(at 3.81 1.92 90)
-			(layer "F.Fab")
+			(at 3.81 0 90)
+			(layer "F.SilkS")
 			(effects
 				(font
@@
 			(at 5.08 0 90)
 			(layer "F.SilkS")
+			(hide yes)
 			(effects
 				(font
@@
 		(property "Value" "1N4004"
 			(at 5.08 2.47 90)
-			(layer "F.Fab")
+			(layer "F.SilkS")
 			(effects
 				(font
@@
 			)
 		)
-		(property "Value" "Water Level"
+		(property "Value" "FLOAT"
 			(at 1.05 5.05 90)
 			(layer "F.SilkS")
@@
 			(at 5.53 0 90)
 			(layer "F.SilkS")
+			(hide yes)
 			(effects
 				(font
@@
 		)
 		(property "Value" "1N4004"
-			(at 5.08 2.47 90)
-			(layer "F.Fab")
+			(at 5.08 2.45 90)
+			(layer "F.SilkS")
 			(effects
 				(font
@@
 			)
 		)
-		(property "Value" "Zone 1"
+		(property "Value" "ZONE 1"
 			(at -4.35 0.45 180)
 			(layer "F.SilkS")
@@
 	(footprint "MountingHole:MountingHole_2.5mm_Pad_TopOnly"
 		(layer "F.Cu")
-		(at 161.55 34.55)
+		(at 161.65 34.65)
 		(descr "Mounting Hole 2.5mm, generated by kicad-footprint-generator mountinghole.py")
 		(tags "mountinghole")
@@
 	)
 	(gr_line
-		(start 196.35 80.05)
-		(end 196.35 25.65)
+		(start 196 80.1)
+		(end 196 25.65)
 		(stroke
 			(width 0.05)
@@
 	)
 	(gr_arc
-		(start 195.8 25.1)
-		(mid 196.188909 25.261091)
-		(end 196.35 25.65)
+		(start 195.45 25.1)
+		(mid 195.838909 25.261091)
+		(end 196 25.65)
 		(stroke
 			(width 0.05)
@@
 	(gr_line
 		(start 121.9 25.1)
-		(end 195.8 25.1)
+		(end 195.45 25.1)
 		(stroke
 			(width 0.05)
@@
 	(gr_line
 		(start 121.9 80.6)
-		(end 195.8 80.6)
+		(end 195.45 80.6)
 		(stroke
 			(width 0.05)
@@
 	)
 	(gr_arc
-		(start 196.35 80.05)
-		(mid 196.188909 80.438909)
-		(end 195.8 80.6)
+		(start 196 80.05)
+		(mid 195.838909 80.438909)
+		(end 195.45 80.6)
 		(stroke
 			(width 0.05)
@@
 		(polygon
 			(pts
-				(xy 121.698646 25.207238) (xy 195.899093 25.457239) (xy 196 80.3) (xy 121.85 80.3)
+				(xy 121.698715 25.232512) (xy 195.399137 25.480827) (xy 195.5 80.3) (xy 122 80.3)
 			)
 		)

Commit message: Fix edge cut
Other:
- board size 74.7 x 55.5 mm -> 75.2 x 55.5 mm
Changed lines of the file:
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@@
 	)
 	(gr_line
-		(start 196 80.1)
-		(end 196 25.65)
+		(start 196.5 80.1)
+		(end 196.5 25.65)
 		(stroke
 			(width 0.05)
@@
 	)
 	(gr_arc
-		(start 195.45 25.1)
-		(mid 195.838909 25.261091)
-		(end 196 25.65)
+		(start 195.95 25.1)
+		(mid 196.338909 25.261091)
+		(end 196.5 25.65)
 		(stroke
 			(width 0.05)
@@
 	(gr_line
 		(start 121.9 25.1)
-		(end 195.45 25.1)
+		(end 195.95 25.1)
 		(stroke
 			(width 0.05)
@@
 	(gr_line
 		(start 121.9 80.6)
-		(end 195.45 80.6)
+		(end 195.95 80.6)
 		(stroke
 			(width 0.05)
@@
 	)
 	(gr_arc
-		(start 196 80.05)
-		(mid 195.838909 80.438909)
-		(end 195.45 80.6)
+		(start 196.5 80.05)
+		(mid 196.338909 80.438909)
+		(end 195.95 80.6)
 		(stroke
 			(width 0.05)
@@
 		(min_thickness 0.25)
 		(filled_areas_thickness no)
-		(fill yes
+		(fill
 			(thermal_gap 0.5)
 			(thermal_bridge_width 0.5)
@@
 		(polygon
 			(pts
-				(xy 121.698715 25.232512) (xy 195.399137 25.480827) (xy 195.5 80.3) (xy 122 80.3)
+				(xy 121.698715 25.232512) (xy 195.89914 25.482512) (xy 196 80.3) (xy 122 80.3)
 			)
 		)
