File: esp32-watering.kicad_pcb (KiCad board)
At the start: 2 copper layers, 75.2 x 55.5 mm, 30 parts, among them J1 12V, J2 DS18B20, J3 FLOAT, J4 PUMP, J5 ZONE 1, J6 ZONE 2, J7 ZONE 3, K1 Pump Control, K2 Zone 1, K3 Zone 2, K4 Zone 3, Q1 2N3904, Q2 2N3904, Q3 2N3904, Q4 2N3904, U1 esp32-wemos-d1-mini, U2 TSR 1-2433

Commit message: V1.2 Change flyback diode location
Parts:
- moved D1 18.5 mm to (185.5, 37.1)
- moved D4 18.5 mm to (185.5, 78.6)
- moved D2 18.5 mm to (185.5, 51.1)
- moved D3 18.5 mm to (185.5, 65.1)
- moved K2 5.50 mm to (174.0, 45.5)
- moved K1 5.50 mm to (174.0, 31.5)
- moved K4 5.05 mm to (174.5, 73.5)
- moved K3 5.00 mm to (174.5, 60.0)
- moved Q3 2.13 mm to (159.5, 57.2)
- moved Q2 1.28 mm to (159.4, 42.7)
- moved Q1 0.58 mm to (159.4, 28.7)
- moved R3 0.20 mm to (156.4, 48.7)
- moved J7 0.06 mm to (192.0, 75.5)
Routing:
- net +12V: track 212.9 -> 197.7 mm
- net Net-(D4-A): track 14.6 -> 29.5 mm
- net Net-(D2-A): track 14.5 -> 28.6 mm
- net Net-(D1-A): track 15.2 -> 27.8 mm
- net Net-(D3-A): track 14.5 -> 26.2 mm
- net Net-(J6-Pin_2): track 6.55 -> 13.2 mm
- net Net-(J4-Pin_2): track 7.06 -> 12.6 mm
- net Net-(J5-Pin_2): track 7.24 -> 12.7 mm
- net Net-(J7-Pin_2): track 7.65 -> 12.4 mm
- net Net-(Q3-B): track 9.24 -> 7.12 mm
- net Net-(Q2-B): track 9.24 -> 7.78 mm
- net Net-(Q1-B): track 8.73 -> 8.04 mm
Other:
- board text added: "ESP32 House Plant Watering Controller Rev 1.2"
- board text removed: "ESP32 House Plant Watering Controller Rev 1.1"

Commit message: Align components, bump version
Parts:
- moved K3 0.50 mm to (174.0, 60.0)
- moved K4 0.50 mm to (174.0, 73.5)
Routing:
- net +12V: track 197.7 -> 199.4 mm
- net Net-(J7-Pin_2): track 12.4 -> 12.9 mm
- net Net-(J6-Pin_2): track 13.2 -> 13.7 mm
Other:
- board text added: "ESP32 House Plant Watering Controller Rev 1.3"
- board text removed: "ESP32 House Plant Watering Controller Rev 1.2"
Changed lines of the file:
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@@
 	(footprint "SR5-12V-200-1C:RELAY_SR5-12V-200-1C"
 		(layer "F.Cu")
-		(at 174.5 73.5)
+		(at 174 73.47)
 		(property "Reference" "K4"
 			(at 0 0 0)
@@
 	(footprint "SR5-12V-200-1C:RELAY_SR5-12V-200-1C"
 		(layer "F.Cu")
-		(at 174.5 60)
+		(at 174 59.97)
 		(property "Reference" "K3"
 			(at 0 0 0)
@@
 		(layer "Edge.Cuts")
 	)
-	(gr_text "ESP32 House Plant \nWatering Controller\nRev 1.2"
+	(gr_text "ESP32 House Plant \nWatering Controller\nRev 1.3"
 		(at 137.9 45 90)
 		(layer "B.SilkS")
@@
 	)
 	(segment
-		(start 170.84 65.66)
-		(end 169.5 67)
+		(start 170.34 77.27)
+		(end 170.34 73.86)
 		(width 1.5)
 		(layer "B.Cu")
@@
 	)
 	(segment
-		(start 170.84 63.8)
-		(end 170.84 65.66)
-		(width 1.5)
-		(layer "B.Cu")
-		(net 1)
-	)
-	(segment
 		(start 168.88 51.08)
 		(end 167.73 52.23)
@@
 	)
 	(segment
-		(start 169.5 67)
-		(end 166 67)
+		(start 173.57 67)
+		(end 174.3 67)
+		(width 1.5)
+		(layer "B.Cu")
+		(net 1)
+	)
+	(segment
+		(start 166 67)
+		(end 174.3 67)
 		(width 1.5)
 		(layer "B.Cu")
@@
 	)
 	(segment
-		(start 170.84 73.36)
-		(end 172.8 71.4)
+		(start 170.34 63.77)
+		(end 173.57 67)
 		(width 1.5)
 		(layer "B.Cu")
@@
 	)
 	(segment
-		(start 169.5 67)
+		(start 174.3 67)
 		(end 177.2 67)
 		(width 1.5)
@@
 	)
 	(segment
-		(start 170.84 77.3)
-		(end 170.84 73.36)
+		(start 192 47)
+		(end 187.92 51.08)
 		(width 1.5)
 		(layer "B.Cu")
@@
 	)
 	(segment
-		(start 192 47)
-		(end 187.92 51.08)
+		(start 170.34 73.86)
+		(end 172.8 71.4)
 		(width 1.5)
 		(layer "B.Cu")
@@
 	)
 	(segment
-		(start 172.1 54.92)
-		(end 170.84 56.18)
+		(start 185.5 54.92)
+		(end 172.1 54.92)
 		(width 0.5)
 		(layer "F.Cu")
@@
 	)
 	(segment
-		(start 185.5 54.92)
+		(start 171.57 54.92)
 		(end 172.1 54.92)
 		(width 0.5)
@@
 	)
 	(segment
-		(start 172.05 68.42)
-		(end 168.8 68.42)
+		(start 170.34 56.15)
+		(end 171.57 54.92)
 		(width 0.5)
 		(layer "F.Cu")
-		(net 5)
+		(net 4)
 	)
 	(segment
-		(start 185.5 68.42)
+		(start 171.57 68.42)
 		(end 172.05 68.42)
 		(width 0.5)
@@
 	)
 	(segment
-		(start 170.84 69.68)
-		(end 172.05 68.47)
+		(start 170.34 69.65)
+		(end 171.57 68.42)
+		(width 0.5)
+		(layer "F.Cu")
+		(net 5)
+	)
+	(segment
+		(start 172.05 68.42)
+		(end 168.8 68.42)
 		(width 0.5)
 		(layer "F.Cu")
@@
 	)
 	(segment
-		(start 172.05 68.47)
+		(start 185.5 68.42)
 		(end 172.05 68.42)
 		(width 0.5)
@@
 	)
 	(segment
-		(start 192 56.55)
-		(end 191.444602 56.55)
+		(start 191.444602 56.55)
+		(end 188.994602 59)
 		(width 1.5)
 		(layer "F.Cu")
@@
 	)
 	(segment
-		(start 191.444602 56.55)
-		(end 188.994602 59)
+		(start 192 56.55)
+		(end 191.444602 56.55)
 		(width 1.5)
 		(layer "F.Cu")
@@
 	)
 	(segment
-		(start 183.82 59)
-		(end 181 56.18)
+		(start 188.994602 59)
+		(end 183.35 59)
 		(width 1.5)
 		(layer "F.Cu")
@@
 	)
 	(segment
-		(start 188.994602 59)
-		(end 183.82 59)
+		(start 183.35 59)
+		(end 180.5 56.15)
 		(width 1.5)
 		(layer "F.Cu")
@@
 	)
 	(segment
-		(start 192 73)
-		(end 184.32 73)
+		(start 183.85 73)
+		(end 180.5 69.65)
 		(width 1.5)
 		(layer "F.Cu")
@@
 	)
 	(segment
-		(start 184.32 73)
-		(end 181 69.68)
+		(start 192 73)
+		(end 183.85 73)
 		(width 1.5)
 		(layer "F.Cu")

Commit message: Extend edge cut
Other:
- board size 75.2 x 55.5 mm -> 75.3 x 55.5 mm
Changed lines of the file:
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@@
 	)
 	(gr_arc
-		(start 121.35 25.65)
-		(mid 121.511091 25.261091)
-		(end 121.9 25.1)
+		(start 121.15 25.65)
+		(mid 121.311091 25.261091)
+		(end 121.7 25.1)
 		(stroke
 			(width 0.05)
@@
 	)
 	(gr_line
-		(start 121.9 25.1)
+		(start 121.7 25.1)
 		(end 195.95 25.1)
 		(stroke
@@
 	)
 	(gr_line
-		(start 121.9 80.6)
+		(start 121.7 80.6)
 		(end 195.95 80.6)
 		(stroke
@@
 	)
 	(gr_line
-		(start 121.35 25.65)
-		(end 121.35 80.05)
+		(start 121.15 25.65)
+		(end 121.15 80.05)
 		(stroke
 			(width 0.05)
@@
 	)
 	(gr_arc
-		(start 121.9 80.6)
-		(mid 121.511091 80.438909)
-		(end 121.35 80.05)
+		(start 121.7 80.6)
+		(mid 121.311091 80.438909)
+		(end 121.15 80.05)
 		(stroke
 			(width 0.05)

Commit message: Submit to manufacture
Parts:
- U1: value esp32-wemos-d1-mini -> ESP32 D1 MINI
Connections:
- R3 pad 2: Net-(U1-IO_32) -> Net-(U1-IO_25)
- R4 pad 2: Net-(U1-IO_12/TDI) -> Net-(U1-IO_32)
- U1 pad 26: unconnected-(U1-IO_25-Pad26) -> Net-(U1-IO_25)
- U1 pad 30: Net-(U1-IO_12/TDI) -> unconnected-(U1-IO_12/TDI-Pad30)
Routing:
- net Net-(U1-IO_12/TDI): track 27.7 -> 0.00 mm
- net Net-(U1-IO_25): track 0.00 -> 21.0 mm
- net Net-(U1-IO_32): track 17.7 -> 29.8 mm
Other:
- board text added: "ESP32 House Plant Watering Controller Rev 1.4"
- board text removed: "ESP32 House Plant Watering Controller Rev 1.3"

Commit message: Bump version, add b.silkscreen for polarity
Other:
- board text added: "+"
- board text added: "-"
- board text added: "D"
- board text added: "ESP32 House Plant Watering Controller Rev 2.1"
- board text removed: "ESP32 House Plant Watering Controller Rev 1.4"
Changed lines of the file:
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@@
 		(layer "Edge.Cuts")
 	)
-	(gr_text "ESP32 House Plant \nWatering Controller\nRev 1.4"
+	(gr_text "-"
+		(at 138.5 71.25 0)
+		(layer "B.SilkS")
+		(effects
+			(font
+				(size 1 1)
+				(thickness 0.12)
+			)
+			(justify left mirror)
+		)
+	)
+	(gr_text "ESP32 House Plant \nWatering Controller\nRev 2.1"
 		(at 137.9 45 90)
 		(layer "B.SilkS")
@@
 		)
 	)
+	(gr_text "+"
+		(at 125.75 71.5 180)
+		(layer "B.SilkS")
+		(effects
+			(font
+				(size 1 1)
+				(thickness 0.12)
+			)
+			(justify left mirror)
+		)
+	)
+	(gr_text "+"
+		(at 141.25 71.25 0)
+		(layer "B.SilkS")
+		(effects
+			(font
+				(size 1 1)
+				(thickness 0.12)
+			)
+			(justify left mirror)
+		)
+	)
+	(gr_text "-"
+		(at 131 71.5 180)
+		(layer "B.SilkS")
+		(effects
+			(font
+				(size 1 1)
+				(thickness 0.12)
+			)
+			(justify left mirror)
+		)
+	)
+	(gr_text "D"
+		(at 128.5 71.5 180)
+		(layer "B.SilkS")
+		(effects
+			(font
+				(size 1 1)
+				(thickness 0.12)
+			)
+			(justify left mirror)
+		)
+	)

Commit message: Bump version, fix manufacturing error
Parts:
- U1: value ESP32 D1 MINI -> esp32-wemos-d1-mini
Connections:
- net Net-(J2-Pin_2) renamed Sensor1
- net Net-(U1-IO_17/D3) renamed Relay3
- net Net-(U1-IO_25) renamed Relay1
- net Net-(U1-IO_27) renamed Relay0
- net Net-(U1-IO_32) renamed Relay2
- J3 pad 1: Net-(J3-Pin_1) -> (no net)
- K1 pad COM_1: Net-(J4-Pin_2) -> unconnected-(K1-PadCOM_1)
- K1 pad COM_2: unconnected-(K1-PadCOM_2) -> GND
- K1 pad NC: GND -> unconnected-(K1-PadNC)
- K1 pad NO: unconnected-(K1-PadNO) -> Net-(J4-Pin_2)
- K2 pad COM_1: Net-(J5-Pin_2) -> unconnected-(K2-PadCOM_1)
- K2 pad COM_2: unconnected-(K2-PadCOM_2) -> GND
- K2 pad NC: GND -> unconnected-(K2-PadNC)
- K2 pad NO: unconnected-(K2-PadNO) -> Net-(J5-Pin_2)
- K3 pad COM_1: Net-(J6-Pin_2) -> unconnected-(K3-PadCOM_1)
- K3 pad COM_2: unconnected-(K3-PadCOM_2) -> GND
- K3 pad NC: GND -> unconnected-(K3-PadNC)
- K3 pad NO: unconnected-(K3-PadNO) -> Net-(J6-Pin_2)
- K4 pad COM_1: Net-(J7-Pin_2) -> unconnected-(K4-PadCOM_1)
- K4 pad COM_2: unconnected-(K4-PadCOM_2) -> GND
- K4 pad NC: GND -> unconnected-(K4-PadNC)
- K4 pad NO: unconnected-(K4-PadNO) -> Net-(J7-Pin_2)
- R1 pad 1: Net-(J3-Pin_1) -> Sensor0
- U1 pad 31: Net-(J3-Pin_1) -> Sensor0
Routing:
- net Sensor0: track 0.00 -> 42.5 mm
- net Net-(J3-Pin_1): track 42.5 -> 0.00 mm
- net Net-(J7-Pin_2): track 12.9 -> 25.6 mm
- net Net-(J5-Pin_2): track 12.7 -> 25.4 mm
- net Net-(J4-Pin_2): track 12.6 -> 25.3 mm
- net Net-(J6-Pin_2): track 13.7 -> 26.4 mm
Other:
- board text added: "ESP32 House Plant Watering Controller Rev 2.2"
- board text removed: "ESP32 House Plant Watering Controller Rev 2.1"
