File: esp32-watering.kicad_sch (KiCad schematic)
At the start: 0 parts

Commit message: Add relays and ESP32
Parts:
- added D1, D2, D3, D4: 1N4004, Diode_THT:D_DO-41_SOD81_P10.16mm_Horizontal, symbol Diode:1N4004
- added J1: 5V, Connector_JST:JST_XH_S2B-XH-A-1_1x02_P2.50mm_Horizontal, symbol Connector:Conn_01x02_Socket
- added J2: 12V, Connector_JST:JST_XH_S2B-XH-A-1_1x02_P2.50mm_Horizontal, symbol Connector:Conn_01x02_Socket
- added K1: Pump Control, SR5-12V-200-1C:RELAY_SR5-12V-200-1C, symbol SR5-12V-200-1C:SR5-12V-200-1C
- added K2: Zone 1, SR5-12V-200-1C:RELAY_SR5-12V-200-1C, symbol SR5-12V-200-1C:SR5-12V-200-1C
- added K3: Zone 2, SR5-12V-200-1C:RELAY_SR5-12V-200-1C, symbol SR5-12V-200-1C:SR5-12V-200-1C
- added K4: Zone 3, SR5-12V-200-1C:RELAY_SR5-12V-200-1C, symbol SR5-12V-200-1C:SR5-12V-200-1C
- added U1: esp32-wemos-d1-mini, esp32-wemos-d1-mini:esp32-wemos-d1-mini, symbol esp32-wemos-d1-mini:esp32-wemos-d1-mini
Connections:
- new net: D2.2 (A), K2.A2
- new net +12V: D1.2 (A), J2.1 (Pin_1), K1.A2
- new net +5V: J1.1 (Pin_1), U1.35 (VCC_(USB))
- new net GND: D1.1 (K), D2.1 (K), D3.1 (K), D4.1 (K), J1.2 (Pin_2), J2.2 (Pin_2), K1.A1, K2.A1, U1.1 (GND), U1.22 (GND), U1.33 (GND)

Commit message: Add pulldown resistor
Parts:
- added J3: Water Level, Connector_JST:JST_XH_B2B-XH-A_1x02_P2.50mm_Vertical, symbol Connector:Conn_01x02_Pin
- added Q1, Q2, Q3, Q4: PN2222A, Package_TO_SOT_THT:TO-92L_HandSolder, symbol Transistor_BJT:PN2222A
- added R1: 10K, symbol Device:R
Connections:
- net +12V: now also D1.1 (K), D2.1 (K), D3.1 (K), D4.1 (K), K2.A2, K3.A2, K4.A2; no longer D1.2 (A)
- net GND: now also R1.1; no longer D1.1 (K), D2.1 (K), D3.1 (K), D4.1 (K), K1.A1, K2.A1
- net at D2.2 (A): now also K2.A1; no longer K2.A2
- new net: D1.2 (A), K1.A1
- new net: J3.2 (Pin_2), R1.2
- new net +3.3V: J3.1 (Pin_1)
Other:
- moved on the sheet: D1, D2, D3, D4

Commit message: First pass of schematic. Three zones.
Parts:
- added J4: Pump, Connector_JST:JST_XH_B2B-XH-A_1x02_P2.50mm_Vertical, symbol Connector:Conn_01x02_Pin
- added J5: Zone 1, Connector_JST:JST_XH_B2B-XH-A_1x02_P2.50mm_Vertical, symbol Connector:Conn_01x02_Pin
- added J6: Zone 2, Connector_JST:JST_XH_B2B-XH-A_1x02_P2.50mm_Vertical, symbol Connector:Conn_01x02_Pin
- added J7: Zone 3, Connector_JST:JST_XH_B2B-XH-A_1x02_P2.50mm_Vertical, symbol Connector:Conn_01x02_Pin
- added R2, R3, R4, R5: 1K6, symbol Device:R
- Q1, Q2, Q3, Q4: value PN2222A -> 2N3904; footprint Package_TO_SOT_THT:TO-92L_HandSolder -> Package_TO_SOT_THT:TO-92_Inline; symbol Transistor_BJT:PN2222A -> Transistor_BJT:2N3904
Connections:
- net +12V: now also J4.1 (Pin_1), J5.1 (Pin_1), J6.1 (Pin_1), J7.1 (Pin_1)
- net GND: now also K1.NC, K2.NC, K3.NC, K4.NC, Q1.1 (E), Q2.1 (E), Q3.1 (E), Q4.1 (E)
- net at D2.2 (A), K2.A1: now also Q2.3 (C)
- net at D3.2 (A): now also K3.A1, Q3.3 (C)
- net at Q1.2 (B): now also R2.1
- net at Q1.3 (C): now also D1.2 (A), K1.A1
- net at Q3.2 (B): now also R4.1
- net at D4.2 (A): now also K4.A1, Q4.3 (C)
- net at K1.COM_1: now also J4.2 (Pin_2)
- net at K3.COM_1: now also J6.2 (Pin_2)
- net at Q4.2 (B): now also R5.1
- net at J3.2 (Pin_2), R1.2: now also U1.24 (IO_27)
- net at Q2.2 (B): now also R3.1
- net at K2.COM_1: now also J5.2 (Pin_2)
- net at K4.COM_1: now also J7.2 (Pin_2)
- net at U1.26 (IO_25): now also R5.2
- net at U1.28 (IO_32): now also R4.2
- net at U1.29 (IO_17/D3): now also R3.2
- net at U1.30 (IO_12/TDI): now also R2.2
Other:
- moved on the sheet: D1, D2, D3, D4, J1, J2, J3, K1, K2, K3, K4, Q1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

Commit message: Start layout
Parts:
- J1, J2: footprint Connector_JST:JST_XH_S2B-XH-A-1_1x02_P2.50mm_Horizontal -> Connector_JST:JST_XH_B2B-XH-A_1x02_P2.50mm_Vertical
- R1, R2, R3, R4, R5: footprint (none) -> Resistor_THT:R_Axial_DIN0204_L3.6mm_D1.6mm_P7.62mm_Horizontal
Changed lines of the file:
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@@
 			)
 		)
-		(property "Footprint" ""
+		(property "Footprint" "Resistor_THT:R_Axial_DIN0204_L3.6mm_D1.6mm_P7.62mm_Horizontal"
 			(at 132.08 74.168 90)
 			(effects
@@
 			)
 		)
-		(property "Footprint" ""
+		(property "Footprint" "Resistor_THT:R_Axial_DIN0204_L3.6mm_D1.6mm_P7.62mm_Horizontal"
 			(at 132.08 51.308 90)
 			(effects
@@
 			)
 		)
-		(property "Footprint" "Connector_JST:JST_XH_S2B-XH-A-1_1x02_P2.50mm_Horizontal"
+		(property "Footprint" "Connector_JST:JST_XH_B2B-XH-A_1x02_P2.50mm_Vertical"
 			(at 209.55 46.99 0)
 			(effects
@@
 			)
 		)
-		(property "Footprint" ""
+		(property "Footprint" "Resistor_THT:R_Axial_DIN0204_L3.6mm_D1.6mm_P7.62mm_Horizontal"
 			(at 132.08 98.298 90)
 			(effects
@@
 			)
 		)
-		(property "Footprint" ""
+		(property "Footprint" "Resistor_THT:R_Axial_DIN0204_L3.6mm_D1.6mm_P7.62mm_Horizontal"
 			(at 132.08 126.238 90)
 			(effects
@@
 			)
 		)
-		(property "Footprint" "Connector_JST:JST_XH_S2B-XH-A-1_1x02_P2.50mm_Horizontal"
+		(property "Footprint" "Connector_JST:JST_XH_B2B-XH-A_1x02_P2.50mm_Vertical"
 			(at 209.55 54.61 0)
 			(effects
@@
 			)
 		)
-		(property "Footprint" ""
+		(property "Footprint" "Resistor_THT:R_Axial_DIN0204_L3.6mm_D1.6mm_P7.62mm_Horizontal"
 			(at 83.058 154.94 90)
 			(effects

Commit message: Initial layout
Connections:
- net +3.3V: now also U1.16 (3V3)
- no-connect marks 0 -> 8
Changed lines of the file:
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@@
 		(color 0 0 0 0)
 	)
+	(no_connect
+		(at 53.34 76.2)
+	)
+	(no_connect
+		(at 53.34 52.07)
+	)
+	(no_connect
+		(at 53.34 100.33)
+	)
+	(no_connect
+		(at 53.34 49.53)
+	)
+	(no_connect
+		(at 53.34 27.94)
+	)
+	(no_connect
+		(at 53.34 25.4)
+	)
+	(no_connect
+		(at 53.34 73.66)
+	)
+	(no_connect
+		(at 53.34 97.79)
+	)
 	(wire
 		(pts
@@
 	(wire
 		(pts
-			(xy 156.21 49.53) (xy 135.89 49.53)
+			(xy 135.89 49.53) (xy 157.48 49.53)
 		)
 		(stroke
@@
 	(wire
 		(pts
-			(xy 156.21 48.26) (xy 157.48 48.26)
-		)
-		(stroke
-			(width 0)
-			(type default)
-		)
-	)
-	(wire
-		(pts
 			(xy 45.72 102.87) (xy 45.72 96.52)
 		)
@@
 	(wire
 		(pts
+			(xy 157.48 49.53) (xy 157.48 102.87)
+		)
+		(stroke
+			(width 0)
+			(type default)
+		)
+	)
+	(wire
+		(pts
 			(xy 71.12 146.05) (xy 71.12 142.24)
 		)
@@
 	(wire
 		(pts
-			(xy 156.21 48.26) (xy 156.21 49.53)
-		)
-		(stroke
-			(width 0)
-			(type default)
-		)
-	)
-	(wire
-		(pts
 			(xy 50.8 59.69) (xy 50.8 62.23)
 		)
@@
 	(wire
 		(pts
+			(xy 195.58 90.17) (xy 217.17 90.17)
+		)
+		(stroke
+			(width 0)
+			(type default)
+		)
+	)
+	(wire
+		(pts
 			(xy 73.66 49.53) (xy 80.01 49.53)
 		)
@@
 	(wire
 		(pts
-			(xy 157.48 48.26) (xy 157.48 102.87)
+			(xy 217.17 90.17) (xy 217.17 87.63)
 		)
 		(stroke
@@
 					(unit 1)
 				)
+			)
+		)
+	)
+	(symbol
+		(lib_id "power:+3.3V")
+		(at 217.17 87.63 0)
+		(unit 1)
+		(exclude_from_sim no)
+		(in_bom yes)
+		(on_board yes)
+		(dnp no)
+		(fields_autoplaced yes)
+		(property "Reference" "#PWR024"
+			(at 217.17 91.44 0)
+			(effects
+				(font
+					(size 1.27 1.27)
+				)
+				(hide yes)
+			)
+		)
+		(property "Value" "+3.3V"
+			(at 217.17 82.55 0)
+			(effects
+				(font
+					(size 1.27 1.27)
+				)
+			)
+		)
+		(property "Footprint" ""
+			(at 217.17 87.63 0)
+			(effects
+				(font
+					(size 1.27 1.27)
+				)
+				(hide yes)
+			)
+		)
+		(property "Datasheet" ""
+			(at 217.17 87.63 0)
+			(effects
+				(font
+					(size 1.27 1.27)
+				)
+				(hide yes)
+			)
+		)
+		(property "Description" "Power symbol creates a global label with name \"+3.3V\""
+			(at 217.17 87.63 0)
+			(effects
+				(font
+					(size 1.27 1.27)
+				)
+				(hide yes)
+			)
+		)
+		(pin "1"
+		)
+		(instances
+			(project ""
+				(path "/2966a4e5-a5f9-4e1b-aa82-21ddf1b5a941"
+					(reference "#PWR024")
+					(unit 1)
+				)

Commit message: Flip float valve
Connections:
- net +3.3V: now also J3.2 (Pin_2); no longer J3.1 (Pin_1)
- net at R1.2, U1.24 (IO_27): now also J3.1 (Pin_1); no longer J3.2 (Pin_2)
Other:
- moved on the sheet: J3
Changed lines of the file:
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@@
 	(wire
 		(pts
-			(xy 64.77 146.05) (xy 71.12 146.05)
-		)
-		(stroke
-			(width 0)
-			(type default)
-		)
-	)
-	(wire
-		(pts
 			(xy 80.01 49.53) (xy 80.01 50.8)
 		)
@@
 	(wire
 		(pts
-			(xy 71.12 146.05) (xy 71.12 142.24)
+			(xy 190.5 46.99) (xy 204.47 46.99)
 		)
 		(stroke
@@
 	(wire
 		(pts
-			(xy 190.5 46.99) (xy 204.47 46.99)
+			(xy 80.01 25.4) (xy 80.01 26.67)
 		)
 		(stroke
@@
 	(wire
 		(pts
-			(xy 80.01 25.4) (xy 80.01 26.67)
+			(xy 210.82 92.71) (xy 210.82 97.79)
 		)
 		(stroke
@@
 	(wire
 		(pts
-			(xy 210.82 92.71) (xy 210.82 97.79)
+			(xy 43.18 81.28) (xy 53.34 81.28)
 		)
 		(stroke
@@
 	(wire
 		(pts
-			(xy 43.18 81.28) (xy 53.34 81.28)
+			(xy 73.66 73.66) (xy 80.01 73.66)
 		)
 		(stroke
@@
 	(wire
 		(pts
-			(xy 73.66 73.66) (xy 80.01 73.66)
+			(xy 50.8 59.69) (xy 50.8 62.23)
 		)
 		(stroke
@@
 	(wire
 		(pts
-			(xy 50.8 59.69) (xy 50.8 62.23)
+			(xy 64.77 151.13) (xy 71.12 151.13)
 		)
 		(stroke
@@
 	(wire
 		(pts
+			(xy 71.12 151.13) (xy 71.12 147.32)
+		)
+		(stroke
+			(width 0)
+			(type default)
+		)
+	)
+	(wire
+		(pts
 			(xy 73.66 25.4) (xy 80.01 25.4)
 		)
@@
 	(symbol
 		(lib_id "power:+3.3V")
-		(at 71.12 142.24 0)
+		(at 71.12 147.32 0)
 		(unit 1)
 		(exclude_from_sim no)
@@
 		(fields_autoplaced yes)
 		(property "Reference" "#PWR010"
-			(at 71.12 146.05 0)
+			(at 71.12 151.13 0)
 			(effects
 				(font
@@
 		)
 		(property "Value" "+3.3V"
-			(at 71.12 137.16 0)
+			(at 71.12 142.24 0)
 			(effects
 				(font
@@
 		)
 		(property "Footprint" ""
-			(at 71.12 142.24 0)
+			(at 71.12 147.32 0)
 			(effects
 				(font
@@
 		)
 		(property "Datasheet" ""
-			(at 71.12 142.24 0)
+			(at 71.12 147.32 0)
 			(effects
 				(font
@@
 		)
 		(property "Description" "Power symbol creates a global label with name \"+3.3V\""
-			(at 71.12 142.24 0)
+			(at 71.12 147.32 0)
 			(effects
 				(font
@@
 	(symbol
 		(lib_id "Connector:Conn_01x02_Pin")
-		(at 59.69 146.05 0)
+		(at 59.69 148.59 0)
 		(unit 1)
 		(exclude_from_sim no)
@@
 		(fields_autoplaced yes)
 		(property "Reference" "J3"
-			(at 60.325 140.97 0)
+			(at 60.325 143.51 0)
 			(effects
 				(font
@@
 		)
 		(property "Value" "Water Level"
-			(at 60.325 143.51 0)
+			(at 60.325 146.05 0)
 			(effects
 				(font
@@
 		)
 		(property "Footprint" "Connector_JST:JST_XH_B2B-XH-A_1x02_P2.50mm_Vertical"
-			(at 59.69 146.05 0)
+			(at 59.69 148.59 0)
 			(effects
 				(font
@@
 		)
 		(property "Datasheet" "~"
-			(at 59.69 146.05 0)
+			(at 59.69 148.59 0)
 			(effects
 				(font
@@
 		)
 		(property "Description" "Generic connector, single row, 01x02, script generated"
-			(at 59.69 146.05 0)
+			(at 59.69 148.59 0)
 			(effects
 				(font

Commit message: Pre-DRC
Connections:
- net at R3.2: now also U1.28 (IO_32); no longer U1.29 (IO_17/D3)
- net at R2.2: now also U1.24 (IO_27); no longer U1.30 (IO_12/TDI)
- net at R4.2: now also U1.30 (IO_12/TDI); no longer U1.28 (IO_32)
- net at R5.2: now also U1.29 (IO_17/D3); no longer U1.26 (IO_25)
- net at J3.1 (Pin_1), R1.2: now also U1.31 (IO_16/D4); no longer U1.24 (IO_27)
- no-connect marks 8 -> 36

Commit message: Add Dallas sensor + decoupling cap
Parts:
- added C1: C_Polarized, symbol Device:C_Polarized
- added J8: DS18B20, Connector_JST:JST_XH_B3B-XH-A_1x03_P2.50mm_Vertical, symbol Connector:Conn_01x03_Pin
- added R6: 4K7, symbol Device:R
Connections:
- net +12V: now also C1.1
- net +3.3V: now also J8.1 (Pin_1), R6.1
- net GND: now also C1.2, J8.3 (Pin_3)
- net at U1.6 (IO_26/D0): now also J8.2 (Pin_2), R6.2
- no-connect marks 36 -> 35
