File: esp32-watering.kicad_sch (KiCad schematic)
At the start: 28 parts, among them J1 5V, J2 12V, J3 Water Level, J4 Pump, J5 Zone 1, J6 Zone 2, J7 Zone 3, J8 DS18B20, K1 Pump Control, K2 Zone 1, K3 Zone 2, K4 Zone 3, Q1 2N3904, Q2 2N3904, Q3 2N3904, Q4 2N3904, U1 esp32-wemos-d1-mini

Commit message: Add Traco 3.3V regulator
Parts:
- removed C1: C_Polarized, symbol Device:C_Polarized
- removed J1: 5V, Connector_JST:JST_XH_B2B-XH-A_1x02_P2.50mm_Vertical, symbol Connector:Conn_01x02_Socket
- added U2: TSR 1-2433, footprints:TSR1-SINGLE_TRP, symbol 2025-10-06_03-42-38:TSR_1-2433
- R6: footprint (none) -> Resistor_THT:R_Axial_DIN0204_L3.6mm_D1.6mm_P7.62mm_Horizontal
- renumbered J2 to J1, J8 to J2
Connections:
- net +12V: now also U2.1 (+VIN)
- net +3.3V: now also J2.3 (Pin_3), R1.2, U2.3 (+VOUT); no longer J2.1 (Pin_1), J3.2 (Pin_2)
- net GND: now also J2.1 (Pin_1), J3.2 (Pin_2), U2.2 (GND); no longer J2.3 (Pin_3), R1.1
- net at J3.1 (Pin_1), U1.31 (IO_16/D4): now also R1.1; no longer R1.2
- net +5V: no longer names the net of U1.35 (VCC_(USB))
- no-connect marks 35 -> 36
Other:
- moved on the sheet: J1, J3, R1

Commit message: Submit to manufacture
Connections:
- net at R3.2: now also U1.26 (IO_25); no longer U1.28 (IO_32)
- net at R4.2: now also U1.28 (IO_32); no longer U1.30 (IO_12/TDI)
Changed lines of the file:
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@@
-	)
-	(no_connect
-		(at 168.91 143.51)
 	)
 	(no_connect
@@
 	)
 	(no_connect
+		(at 168.91 102.87)
+	)
+	(no_connect
 		(at 168.91 95.25)
 	)
@@
 	(wire
 		(pts
+			(xy 165.1 120.65) (xy 168.91 120.65)
+		)
+		(stroke
+			(width 0)
+			(type default)
+		)
+	)
+	(wire
+		(pts
 			(xy 53.34 59.69) (xy 50.8 59.69)
 		)
@@
 	(wire
 		(pts
+			(xy 168.91 143.51) (xy 163.83 143.51)
+		)
+		(stroke
+			(width 0)
+			(type default)
+		)
+	)
+	(wire
+		(pts
 			(xy 252.73 46.99) (xy 254 46.99)
 		)
@@
 	(wire
 		(pts
-			(xy 135.89 96.52) (xy 161.29 96.52)
-		)
-		(stroke
-			(width 0)
-			(type default)
-		)
-	)
-	(wire
-		(pts
-			(xy 161.29 96.52) (xy 161.29 102.87)
+			(xy 135.89 96.52) (xy 165.1 96.52)
+		)
+		(stroke
+			(width 0)
+			(type default)
+		)
+	)
+	(wire
+		(pts
+			(xy 165.1 96.52) (xy 165.1 120.65)
 		)
 		(stroke
@@
 	(wire
 		(pts
+			(xy 163.83 127) (xy 154.94 127)
+		)
+		(stroke
+			(width 0)
+			(type default)
+		)
+	)
+	(wire
+		(pts
 			(xy 73.66 83.82) (xy 80.01 83.82)
 		)
@@
 	(wire
 		(pts
-			(xy 154.94 72.39) (xy 154.94 120.65)
+			(xy 154.94 72.39) (xy 154.94 127)
 		)
 		(stroke
@@
 	(wire
 		(pts
-			(xy 154.94 120.65) (xy 168.91 120.65)
-		)
-		(stroke
-			(width 0)
-			(type default)
-		)
-	)
-	(wire
-		(pts
 			(xy 195.58 95.25) (xy 195.58 97.79)
 		)
@@
 	(wire
 		(pts
-			(xy 161.29 102.87) (xy 168.91 102.87)
-		)
-		(stroke
-			(width 0)
-			(type default)
-		)
-	)
-	(wire
-		(pts
 			(xy 106.68 72.39) (xy 128.27 72.39)
 		)
@@
 		)
 		(stroke
+			(width 0)
+			(type default)
+		)
+	)
+	(wire
+		(pts
+			(xy 163.83 143.51) (xy 163.83 127)
+		)
+		(stroke

Commit message: Name nets
Connections:
- net Relay1: now reaches R3.2, U1.26 (IO_25)
- net Relay0: now reaches R2.2, U1.24 (IO_27)
- net Relay2: now reaches R4.2, U1.28 (IO_32)
- net Sensor1: now reaches J2.2 (Pin_2), R6.2, U1.6 (IO_26/D0)
- net Relay3: now reaches R5.2, U1.29 (IO_17/D3)
- net Sensor0: now reaches J3.1 (Pin_1), R1.1, U1.31 (IO_16/D4)
Other:
- note added: "POWER"
- note added: "SENSORS"
- moved on the sheet: J2, J3, R1, R6, U1

Commit message: Bump version, fix manufacturing error
Connections:
- net GND: now also K1.COM_2, K2.COM_2, K3.COM_2, K4.COM_2; no longer K1.NC, K2.NC, K3.NC, K4.NC
- net at J5.2 (Pin_2): now also K2.NO; no longer K2.COM_1
- net at K1.COM_1: no longer J4.2 (Pin_2)
- net at K1.NO: now also J4.2 (Pin_2)
- net at K3.COM_1: no longer J6.2 (Pin_2)
- net at K3.NO: now also J6.2 (Pin_2)
- net at J7.2 (Pin_2): now also K4.NO; no longer K4.COM_1
Changed lines of the file:
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@@
 	)
 	(no_connect
-		(at 53.34 76.2)
-	)
-	(no_connect
-		(at 53.34 52.07)
-	)
-	(no_connect
-		(at 53.34 100.33)
-	)
-	(no_connect
-		(at 53.34 49.53)
-	)
-	(no_connect
-		(at 53.34 27.94)
+		(at 53.34 57.15)
 	)
 	(no_connect
@@
 	)
 	(no_connect
-		(at 53.34 25.4)
-	)
-	(no_connect
 		(at 246.38 104.14)
 	)
 	(no_connect
+		(at 53.34 83.82)
+	)
+	(no_connect
 		(at 246.38 129.54)
 	)
 	(no_connect
+		(at 53.34 59.69)
+	)
+	(no_connect
 		(at 219.71 129.54)
 	)
@@
 	)
 	(no_connect
+		(at 53.34 105.41)
+	)
+	(no_connect
 		(at 219.71 109.22)
 	)
@@
 	)
 	(no_connect
-		(at 53.34 73.66)
+		(at 53.34 81.28)
+	)
+	(no_connect
+		(at 53.34 35.56)
 	)
 	(no_connect
@@
 	)
 	(no_connect
+		(at 53.34 107.95)
+	)
+	(no_connect
 		(at 219.71 119.38)
 	)
 	(no_connect
+		(at 53.34 33.02)
+	)
+	(no_connect
 		(at 219.71 106.68)
 	)
@@
 	)
 	(no_connect
-		(at 53.34 97.79)
-	)
-	(no_connect
 		(at 219.71 132.08)
 	)
@@
 	(wire
 		(pts
+			(xy 48.26 33.02) (xy 48.26 25.4)
+		)
+		(stroke
+			(width 0)
+			(type default)
+		)
+	)
+	(wire
+		(pts
 			(xy 80.01 107.95) (xy 80.01 106.68)
 		)
@@
 	(wire
 		(pts
-			(xy 53.34 59.69) (xy 50.8 59.69)
+			(xy 50.8 27.94) (xy 53.34 27.94)
+		)
+		(stroke
+			(width 0)
+			(type default)
+		)
+	)
+	(wire
+		(pts
+			(xy 53.34 100.33) (xy 50.8 100.33)
 		)
 		(stroke
@@
 	(wire
 		(pts
+			(xy 43.18 33.02) (xy 48.26 33.02)
+		)
+		(stroke
+			(width 0)
+			(type default)
+		)
+	)
+	(wire
+		(pts
 			(xy 118.11 35.56) (xy 118.11 38.1)
 		)
@@
 	(wire
 		(pts
+			(xy 48.26 81.28) (xy 48.26 73.66)
+		)
+		(stroke
+			(width 0)
+			(type default)
+		)
+	)
+	(wire
+		(pts
 			(xy 118.11 163.83) (xy 121.92 163.83)
 		)
@@
 	(wire
 		(pts
+			(xy 48.26 57.15) (xy 48.26 49.53)
+		)
+		(stroke
+			(width 0)
+			(type default)
+		)
+	)
+	(wire
+		(pts
 			(xy 111.76 35.56) (xy 118.11 35.56)
 		)
@@
 	(wire
 		(pts
-			(xy 50.8 83.82) (xy 50.8 86.36)
+			(xy 50.8 76.2) (xy 50.8 86.36)
 		)
 		(stroke
@@
 	(wire
 		(pts
+			(xy 48.26 105.41) (xy 48.26 97.79)
+		)
+		(stroke
+			(width 0)
+			(type default)
+		)
+	)
+	(wire
+		(pts
 			(xy 252.73 46.99) (xy 254 46.99)
 		)
@@
 	(wire
 		(pts
-			(xy 43.18 33.02) (xy 53.34 33.02)
-		)
-		(stroke
-			(width 0)
-			(type default)
-		)
-	)
-	(wire
-		(pts
 			(xy 80.01 35.56) (xy 101.6 35.56)
 		)
@@
 	(wire
 		(pts
+			(xy 48.26 25.4) (xy 53.34 25.4)
+		)
+		(stroke
+			(width 0)
+			(type default)
+		)
+	)
+	(wire
+		(pts
 			(xy 106.68 91.44) (xy 106.68 96.52)
 		)
@@
 	(wire
 		(pts
-			(xy 53.34 107.95) (xy 50.8 107.95)
-		)
-		(stroke
-			(width 0)
-			(type default)
-		)
-	)
-	(wire
-		(pts
-			(xy 53.34 35.56) (xy 50.8 35.56)
+			(xy 43.18 105.41) (xy 48.26 105.41)
 		)
 		(stroke
@@
 	(wire
 		(pts
-			(xy 43.18 81.28) (xy 53.34 81.28)
-		)
-		(stroke
-			(width 0)
-			(type default)
-		)
-	)
-	(wire
-		(pts
 			(xy 73.66 73.66) (xy 80.01 73.66)
 		)
@@
 	(wire
 		(pts
-			(xy 50.8 59.69) (xy 50.8 62.23)
-		)
-		(stroke
-			(width 0)
-			(type default)
-		)
-	)
-	(wire
-		(pts
 			(xy 73.66 83.82) (xy 80.01 83.82)
 		)
@@
 	(wire
 		(pts
+			(xy 50.8 76.2) (xy 53.34 76.2)
+		)
+		(stroke
+			(width 0)
+			(type default)
+		)
+	)
+	(wire
+		(pts
 			(xy 118.11 107.95) (xy 118.11 110.49)
 		)
@@
 	(wire
 		(pts
+			(xy 48.26 49.53) (xy 53.34 49.53)
+		)
+		(stroke
+			(width 0)
+			(type default)
+		)
+	)
+	(wire
+		(pts
+			(xy 53.34 52.07) (xy 50.8 52.07)
+		)
+		(stroke
+			(width 0)
+			(type default)
+		)
+	)
+	(wire
+		(pts
 			(xy 111.76 83.82) (xy 118.11 83.82)
 		)
@@
 	(wire
 		(pts
-			(xy 43.18 57.15) (xy 53.34 57.15)
-		)
-		(stroke
-			(width 0)
-			(type default)
-		)
-	)
-	(wire
-		(pts
 			(xy 106.68 96.52) (xy 128.27 96.52)
 		)
@@
 	(wire
 		(pts
-			(xy 50.8 35.56) (xy 50.8 38.1)
+			(xy 50.8 27.94) (xy 50.8 38.1)
 		)
 		(stroke
@@
 	(wire
 		(pts
-			(xy 53.34 83.82) (xy 50.8 83.82)
-		)
-		(stroke
-			(width 0)
-			(type default)
-		)
-	)
-	(wire
-		(pts
-			(xy 50.8 107.95) (xy 50.8 110.49)
+			(xy 50.8 100.33) (xy 50.8 110.49)
 		)
 		(stroke
@@
 	(wire
 		(pts
+			(xy 43.18 81.28) (xy 48.26 81.28)
+		)
+		(stroke
+			(width 0)
+			(type default)
+		)
+	)
+	(wire
+		(pts
 			(xy 43.18 78.74) (xy 45.72 78.74)
 		)
@@
 	(wire
 		(pts
+			(xy 43.18 57.15) (xy 48.26 57.15)
+		)
+		(stroke
+			(width 0)
+			(type default)
+		)
+	)
+	(wire
+		(pts
 			(xy 73.66 35.56) (xy 80.01 35.56)
 		)
@@
 	(wire
 		(pts
+			(xy 50.8 52.07) (xy 50.8 62.23)
+		)
+		(stroke
+			(width 0)
+			(type default)
+		)
+	)
+	(wire
+		(pts
 			(xy 78.74 168.91) (xy 85.09 168.91)
 		)
@@
 	(wire
 		(pts
-			(xy 43.18 105.41) (xy 53.34 105.41)
+			(xy 48.26 73.66) (xy 53.34 73.66)
 		)
 		(stroke
@@
 		)
 		(stroke
+			(width 0)
+			(type default)
+		)
+	)
+	(wire
+		(pts
+			(xy 48.26 97.79) (xy 53.34 97.79)
+		)
+		(stroke
